Commit message: Temp - set hard coded TF for workcell-teststand xacro with new assumption we are defining base_link to workcell

File: src/picknik_ur_bin_picking_config/description/workcell-teststand.xacro (robot description, xacro)
@@ -38,5 +38,5 @@
       <parent link="${parent_link}"/>
       <child link="workcell"/>
-      <origin rpy="0 0 0" xyz="0 0 0"/>
+      <origin xyz="0.026 0.280 0.200" rpy="0 0 ${-pi/2}"/>
     </joint>
     <joint name="workcell_to_robot_mount" type="fixed">
